File: wiring/main/main.kicad_sch (KiCad schematic)
At the start: 14 parts

Commit message: basic implémentation of the last commit
Parts:
- removed A1: Arduino_Nano_v2.x, Module:Arduino_Nano, symbol MCU_Module:Arduino_Nano_v2.x
- added STM32: STM32F042K6Tx, Package_QFP:LQFP-32_7x7mm_P0.8mm, symbol MCU_ST_STM32F0:STM32F042K6Tx
- gave numbers to parts that had none: 13
Connections:
- net +3.3V: now also STM32.1 (VDD)
- net GND: now also RV1.1, STM32.16 (VSS)
- net LEDs: now also STM32.26 (PB3)
- net at D6.1 (K): now also STM32.29 (PB6)
- net at D2.1 (K): now also STM32.27 (PB4)
- net at D4.1 (K): now also STM32.28 (PB5)
- net +5V: now reaches D1.2 (A), D3.2 (A), D5.2 (A), RV1.3
